Commit message: feat(perceptive_grasp): unify hardware simulation and voice
Signed-off-by: wangjie <jie.wang@spacemit.com>

File: perceptive_grasp/urdf/so101.urdf (robot description, URDF)
Before this commit: robot so101, 8 links, 7 joints
Links:
- added link linksee_gripper_tcp_link, mass 1e-9
Joints:
- added joint linksee_gripper_tcp_joint: type fixed, parent gripper_link, child linksee_gripper_tcp_link, origin xyz=0.020 0.016 -0.088 rpy=0 3.14159 0
